File: Kicad/TeleInfoSTM32WB/TeleInfoSTM32WB.sch (KiCad schematic (older format))
At the start: 34 parts, among them J1 Conn_01x02_Female, J2 Conn_01x05_Female, J3 RSP-122811-01, J4 Conn_01x05_Female, SW1 SW_Push, U1 STM32WB55CCUx, U2 SFH620A-1, U3 LM2937-IMP, Y1 32.768 KHz, Y2 Crystal_GND24

Commit message: PCB V6 (forget commited filed.... :clap:)
Parts:
- removed AE1: MLPF-WB55-01E3, MLPF-WB55-01E3:MLPF-WB55-01E3, symbol MLPF-WB55-01E3:MLPF-WB55-01E3
- removed C8: 470mF, Capacitor_SMD:C_Elec_10x10.2, symbol Device:C
- removed D4: LED, LED_SMD:LED_0805_2012Metric_Pad1.15x1.40mm_HandSolder, symbol Device:LED
- removed J1: Conn_01x02_Female, Connector_PinHeader_2.54mm:PinHeader_1x02_P2.54mm_Vertical, symbol Connector:Conn_01x02_Female
- removed JP1: Jumper_3_Open, Jumper:SolderJumper-3_P1.3mm_Open_Pad1.0x1.5mm, symbol Jumper:Jumper_3_Open
- removed R1: 10K, Resistor_SMD:R_0805_2012Metric_Pad1.20x1.40mm_HandSolder, symbol Device:R
- removed R4: 100K, Resistor_SMD:R_0805_2012Metric_Pad1.20x1.40mm_HandSolder, symbol Device:R
- removed R5: R750, Resistor_SMD:R_0805_2012Metric_Pad1.20x1.40mm_HandSolder, symbol Device:R
- added 4.7K1: R, Resistor_SMD:R_0805_2012Metric, symbol Device:R
- added C11: 0.3pF, Capacitor_SMD:C_0805_2012Metric_Pad1.18x1.45mm_HandSolder, symbol Device:C
- added C12, C13, C14, C15, C16, C18, C20: 100nF, Capacitor_SMD:C_0805_2012Metric_Pad1.18x1.45mm_HandSolder, symbol Device:C
- added C17, C19: 4.7uF, Capacitor_SMD:C_0805_2012Metric_Pad1.18x1.45mm_HandSolder, symbol Device:C
- added D4: D, Diode_SMD:D_SOD-123F, symbol Device:D
- added FL1: 2450LP14B100T, Customs:2450LP14B100T, symbol 2450LP14B100T:2450LP14B100T
- added J1: Conn_01x02_Male, Connector_PinHeader_2.54mm:PinHeader_1x02_P2.54mm_Vertical, symbol Connector:Conn_01x02_Male
- added J5: USB_B_Micro, Connector_USB:USB_Micro-B_Molex_47346-0001, symbol Connector:USB_B_Micro
- added L1: 2.7nH, Inductor_SMD:L_0603_1608Metric_Pad1.05x0.95mm_HandSolder, symbol pspice:INDUCTOR
- added L2: Z0603C601ASMST, Inductor_SMD:L_0603_1608Metric_Pad1.05x0.95mm_HandSolder, symbol Device:L_Core_Ferrite
- added L3, L4: 10nH, Inductor_SMD:L_0805_2012Metric, symbol pspice:INDUCTOR
- added SW2: SW_SPDT, Button_Switch_SMD:SW_SPDT_CK-JS102011SAQN, symbol Switch:SW_SPDT
- C5: value 100nF -> 0.8pF; LCSC C138340 -> C464454
- D1: value BAT54H -> D; LCSC C475620 -> (none)
Connections:
- net +3V3: now also U1.1 (VBAT), U1.34 (VDDSMPS), U1.40 (VDDUSB), 4.7K1.2, C12.1, C13.1, C14.1, C16.1, C17.1, C18.1, L2.1; no longer U1.8 (VDDA)
- net +5V: now also D4.2 (A), J5.1 (VBUS)
- net GND: now also C5.2, SW1.2, U1.49 (Pad), C11.2, C12.2, C13.2, C14.2, C15.2, C16.2, C17.2, C18.2, C19.2, C20.2, FL1.1 (GND_1), FL1.3 (GND_2), FL1.4 (GND_3), FL1.6 (GND_4), J5.5 (GND), J5.6 (Shield), SW2.1 (A); no longer C5.1, SW1.1
- net NRST: now also SW1.1, U1.7 (NRST), C20.1; no longer D1.1 (K)
- net at U1.14 (PA5): now also R2.2
- net BT_UART_TX: now reaches U1.18 (PA9)
- net BT_UART_TX: now also J1.2 (Pin_2)
- net at U1.21 (RF1): now also C5.1, L1.1
- net at U1.28 (PB0): now also R3.2
- net VFBFMPS: now reaches U1.31 (VFBSMPS)
- net VFBFMPS: now also C19.1, L3.2
- net VLXSMPS: now reaches U1.33 (VLXSMPS)
- net VLXSMPS: now also L4.1
- net BT_UART_RX: now reaches U1.36 (PA10)
- net BT_UART_RX: now also J1.1 (Pin_1)
- net USB_DM: now reaches U1.37 (PA11)
- net USB_DM: now also J5.2 (D-); no longer SW1.2
- net USB_DP: now reaches U1.38 (PA12)
- net USB_DP: now also J5.3 (D+)
- net at U1.4 (PH3-BOOT0): now also SW2.2 (B)
- net at U1.45 (PB5): no longer R3.2
- net at U1.47 (PB7): no longer R2.2
- net at J3.1: now also FL1.5 (OUT)
- net at C6.1, C7.1, D5.2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: now also D1.2 (A)
- net at C9.2, U3.1 (VI): now also D1.1 (K), D4.1 (K)
- new net: C11.1, FL1.2 (IN), L1.2
- new net: L3.1, L4.2
- new net: 4.7K1.1, SW2.3 (C)
- new net VDDA: C15.1, L2.2, U1.8 (VDDA)
- no-connect marks 0 -> 18
Other:
- note added: "Antenna"
- moved on the sheet: C1, C4, C6, C7, D2, D3, D5, D6, J3, R2, R3, SW1

Commit message: Update symbol stm32wb55
Parts:
- U1: symbol STM32CUBE:STM32WB55CCUx -> stm32:STM32WB55CCUx
Changed lines of the file:
@@
 $EndComp
 $Comp
-L STM32CUBE:STM32WB55CCUx U1
+L stm32:STM32WB55CCUx U1
 U 1 1 610AD110
 P 4800 4350
